Commit message: Add five-point physical table calibration workflow

File: src/dual_crx_description/urdf/dual_crx.urdf.xacro (robot description, xacro)
@@ -7,10 +7,16 @@
   <xacro:include filename="$(find fanuc_crx_description)/urdf/crx5ia_urdf_macro.xacro"/>
   <link name="world"/>
+  <link name="table_frame"/>
+  <joint name="world_to_table" type="fixed">
+    <origin xyz="0 0 0" rpy="0 0 0"/>
+    <parent link="world"/>
+    <child link="table_frame"/>
+  </joint>
   <link name="left_ee_mount"/>
-  <xacro:crx5ia prefix="left_" parent="world" child="left_ee_mount">
+  <xacro:crx5ia prefix="left_" parent="table_frame" child="left_ee_mount">
     <origin xyz="$(arg left_xyz)" rpy="$(arg left_rpy)"/>
   </xacro:crx5ia>
   <link name="right_ee_mount"/>
-  <xacro:crx5ia prefix="right_" parent="world" child="right_ee_mount">
+  <xacro:crx5ia prefix="right_" parent="table_frame" child="right_ee_mount">
     <origin xyz="$(arg right_xyz)" rpy="$(arg right_rpy)"/>
   </xacro:crx5ia>

Commit message: Add frame-aware GUI and five-point verification

File: src/dual_crx_description/urdf/dual_crx.urdf.xacro (robot description, xacro)
@@ -5,4 +5,5 @@
   <xacro:arg name="right_xyz" default="0.0 -0.3 0.0"/>
   <xacro:arg name="right_rpy" default="0.0 0.0 0.0"/>
+  <xacro:arg name="table_collision_size" default="0.30"/>
   <xacro:include filename="$(find fanuc_crx_description)/urdf/crx5ia_urdf_macro.xacro"/>
   <link name="world"/>
@@ -12,4 +13,26 @@
     <parent link="world"/>
     <child link="table_frame"/>
+  </joint>
+  <link name="calibration_table_surface">
+    <visual>
+      <origin xyz="0 0 -0.02" rpy="0 0 0"/>
+      <geometry>
+        <box size="$(arg table_collision_size) $(arg table_collision_size) 0.04"/>
+      </geometry>
+      <material name="calibration_table_gray">
+        <color rgba="0.45 0.45 0.45 0.45"/>
+      </material>
+    </visual>
+    <collision>
+      <origin xyz="0 0 -0.02" rpy="0 0 0"/>
+      <geometry>
+        <box size="$(arg table_collision_size) $(arg table_collision_size) 0.04"/>
+      </geometry>
+    </collision>
+  </link>
+  <joint name="table_to_calibration_surface" type="fixed">
+    <parent link="table_frame"/>
+    <child link="calibration_table_surface"/>
+    <origin xyz="0 0 0" rpy="0 0 0"/>
   </joint>
   <link name="left_ee_mount"/>

File: src/dual_crx_moveit_config/config/dual_crx.urdf.xacro (robot description, xacro)
@@ -5,4 +5,5 @@
   <xacro:arg name="right_xyz" default="0.0 -0.3 0.0"/>
   <xacro:arg name="right_rpy" default="0.0 0.0 0.0"/>
+  <xacro:arg name="table_collision_size" default="0.30"/>
   <xacro:include filename="$(find fanuc_crx_description)/urdf/crx5ia_urdf_macro.xacro"/>
   <link name="world"/>
@@ -12,4 +13,27 @@
     <parent link="world"/>
     <child link="table_frame"/>
+  </joint>
+  <!-- Protect the calibrated five-point area. The box top is table Z=0. -->
+  <link name="calibration_table_surface">
+    <visual>
+      <origin xyz="0 0 -0.02" rpy="0 0 0"/>
+      <geometry>
+        <box size="$(arg table_collision_size) $(arg table_collision_size) 0.04"/>
+      </geometry>
+      <material name="calibration_table_gray">
+        <color rgba="0.45 0.45 0.45 0.45"/>
+      </material>
+    </visual>
+    <collision>
+      <origin xyz="0 0 -0.02" rpy="0 0 0"/>
+      <geometry>
+        <box size="$(arg table_collision_size) $(arg table_collision_size) 0.04"/>
+      </geometry>
+    </collision>
+  </link>
+  <joint name="table_to_calibration_surface" type="fixed">
+    <parent link="table_frame"/>
+    <child link="calibration_table_surface"/>
+    <origin xyz="0 0 0" rpy="0 0 0"/>
   </joint>
   <link name="left_ee_mount"/>
